File: kicad/rc_power_sockets.sch (KiCad schematic (older format))
At the start: 18 parts, among them IC1 ATTINY85-S, J1 Motion Sensor, J2 Radio 433MHZ, P1 ICSP, Q1 N-Channel Mosfet, Q2 P-Channel Mosfet, SW1 Power Switch, U1 LDO 3v3 Voltage Regulator

Commit message: Use existing parts
Parts:
- removed Q1: N-Channel Mosfet, TO_SOT_Packages_SMD:SOT-23_Handsoldering, symbol Q_NPN_BCE
- removed Q2: P-Channel Mosfet, TO_SOT_Packages_SMD:SOT-23_Handsoldering, symbol BC808-40
- removed U1: LDO 3v3 Voltage Regulator, TO_SOT_Packages_SMD:SOT-23_Handsoldering, symbol APE8865N-33-HF-3
- added Q1: Q_NMOS_GSD, TO_SOT_Packages_SMD:SOT-23_Handsoldering, symbol Q_NMOS_GSD
- added Q2: Q_PMOS_GSD, TO_SOT_Packages_SMD:SOT-23_Handsoldering, symbol Q_PMOS_GSD
- added R5: 100K, Resistors_SMD:R_0805_HandSoldering, symbol R
- added RV1: POT, Potentiometers:Potentiometer_WirePads_largePads, symbol POT
- added U1: MCP1700T-3302E/TT, TO_SOT_Packages_SMD:SOT-23_Handsoldering, symbol APE8865N-12-HF-3
- C1, C2, C3: footprint Capacitors_SMD:C_1206_HandSoldering -> Capacitors_SMD:C_0805_HandSoldering
- D1, D2: footprint SMD_Packages:SMD-1206_Pol -> Diodes_SMD:SOD-123
- R1, R2, R3, R4: footprint Resistors_SMD:R_1206_HandSoldering -> Resistors_SMD:R_0805_HandSoldering
- SW1: footprint Buttons_Switches_ThroughHole:SW_Micro_SPST_Angled -> Buttons_Switches_ThroughHole:SW_Micro_SPST
Connections:
- net GND: now also Q1.2 (S), R5.2, U1.1 (GND)
- net at R2.2: now also Q1.3 (D), Q2.1 (G)
- net at C1.1, J2.3: now also Q2.2 (S), U1.3 (VIN)
- net at J1.3, JP1.1, R2.1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: now also Q2.3 (D)
- net at R1.1, R3.1: now also Q1.1 (G)
- net at C2.1, C3.1, IC1.8 (VCC)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: now also RV1.3, U1.2 (VOUT)
- net ADC3: now reaches IC1.2 (PB3(XTAL1/CLKI/OC1B/ADC3/PCINT3))
- net ADC3: now also RV1.2
- net +BATT renamed VCC
- new net: R5.1, RV1.1
Changed lines of the file:
@@
 $EndDescr
-$Comp
-L BC808-40 Q2
-U 1 1 56D4AD58
-P 6450 2450
-F 0 "Q2" H 6650 2525 50  0000 L CNN
-F 1 "P-Channel Mosfet" H 6650 2450 50  0000 L CNN
-F 2 "TO_SOT_Packages_SMD:SOT-23_Handsoldering" H 6650 2375 50  0000 L CIN
-F 3 "" H 6450 2450 50  0000 L CNN
-	1    6450 2450
-	1    0    0    -1
-$EndComp
-$Comp
-L Q_NPN_BCE Q1
-U 1 1 56D4ADA3
-P 5450 3150
-F 0 "Q1" H 5750 3200 50  0000 R CNN
-F 1 "N-Channel Mosfet" H 6350 3100 50  0000 R CNN
-F 2 "TO_SOT_Packages_SMD:SOT-23_Handsoldering" H 5650 3250 50  0001 C CNN
-F 3 "" H 5450 3150 50  0000 C CNN
-	1    5450 3150
-	1    0    0    -1
-$EndComp
-$Comp
-L +BATT #PWR01
-U 1 1 56D4AEA2
-P 6800 1050
-F 0 "#PWR01" H 6800 900 50  0001 C CNN
-F 1 "+BATT" H 6800 1190 50  0000 C CNN
-F 2 "" H 6800 1050 50  0000 C CNN
-F 3 "" H 6800 1050 50  0000 C CNN
-	1    6800 1050
-	1    0    0    -1
-$EndComp
 $Comp
 L R R1
@@
 F 0 "R1" V 4880 3150 50  0000 C CNN
 F 1 "200" V 4800 3150 50  0000 C CNN
-F 2 "Resistors_SMD:R_1206_HandSoldering" V 4730 3150 50  0001 C CNN
+F 2 "Resistors_SMD:R_0805_HandSoldering" V 4730 3150 50  0001 C CNN
 F 3 "" H 4800 3150 50  0000 C CNN
 	1    4800 3150
@@
 F 0 "R2" V 5630 2250 50  0000 C CNN
 F 1 "100K" V 5550 2250 50  0000 C CNN
-F 2 "Resistors_SMD:R_1206_HandSoldering" V 5480 2250 50  0001 C CNN
+F 2 "Resistors_SMD:R_0805_HandSoldering" V 5480 2250 50  0001 C CNN
 F 3 "" H 5550 2250 50  0000 C CNN
 	1    5550 2250
@@
 $EndComp
 $Comp
-L GND #PWR02
+L GND #PWR01
 U 1 1 56D4B298
 P 7350 4400
-F 0 "#PWR02" H 7350 4150 50  0001 C CNN
+F 0 "#PWR01" H 7350 4150 50  0001 C CNN
 F 1 "GND" H 7350 4250 50  0000 C CNN
 F 2 "" H 7350 4400 50  0000 C CNN
@@
 $EndComp
 $Comp
-L GND #PWR03
+L GND #PWR02
 U 1 1 56D4D563
 P 5550 3800
-F 0 "#PWR03" H 5550 3550 50  0001 C CNN
+F 0 "#PWR02" H 5550 3550 50  0001 C CNN
 F 1 "GND" H 5550 3650 50  0000 C CNN
 F 2 "" H 5550 3800 50  0000 C CNN
@@
 F 0 "C2" H 8025 4100 50  0000 L CNN
 F 1 "10uf" H 8025 3900 50  0000 L CNN
-F 2 "Capacitors_SMD:C_1206_HandSoldering" H 8038 3850 50  0001 C CNN
+F 2 "Capacitors_SMD:C_0805_HandSoldering" H 8038 3850 50  0001 C CNN
 F 3 "" H 8000 4000 50  0000 C CNN
 	1    8000 4000
-	1    0    0    -1
-$EndComp
-$Comp
-L APE8865N-33-HF-3 U1
-U 1 1 56D4DF04
-P 7350 3900
-F 0 "U1" H 7100 3650 50  0000 C CNN
-F 1 "LDO 3v3 Voltage Regulator" H 7350 4100 50  0000 C CNN
-F 2 "TO_SOT_Packages_SMD:SOT-23_Handsoldering" H 7350 4000 50  0000 C CIN
-F 3 "" H 7350 3900 50  0000 C CNN
-	1    7350 3900
 	1    0    0    -1
 $EndComp
@@
 F 0 "C1" H 6725 4100 50  0000 L CNN
 F 1 "10uf" H 6725 3900 50  0000 L CNN
-F 2 "Capacitors_SMD:C_1206_HandSoldering" H 6738 3850 50  0001 C CNN
+F 2 "Capacitors_SMD:C_0805_HandSoldering" H 6738 3850 50  0001 C CNN
 F 3 "" H 6700 4000 50  0000 C CNN
 	1    6700 4000
@@
 $EndComp
 $Comp
-L GND #PWR04
+L GND #PWR03
 U 1 1 56D4E393
 P 7600 5550
-F 0 "#PWR04" H 7600 5300 50  0001 C CNN
+F 0 "#PWR03" H 7600 5300 50  0001 C CNN
 F 1 "GND" H 7600 5400 50  0000 C CNN
 F 2 "" H 7600 5550 50  0000 C CNN
@@
 F 0 "D1" H 4150 3000 50  0000 C CNN
 F 1 "D" H 4150 2800 50  0000 C CNN
-F 2 "SMD_Packages:SMD-1206_Pol" H 4150 2900 50  0001 C CNN
+F 2 "Diodes_SMD:SOD-123" H 4150 2900 50  0001 C CNN
 F 3 "" H 4150 2900 50  0000 C CNN
 	1    4150 2900
@@
 F 0 "D2" H 4150 3550 50  0000 C CNN
 F 1 "D" H 4150 3350 50  0000 C CNN
-F 2 "SMD_Packages:SMD-1206_Pol" H 4150 3450 50  0001 C CNN
+F 2 "Diodes_SMD:SOD-123" H 4150 3450 50  0001 C CNN
 F 3 "" H 4150 3450 50  0000 C CNN
 	1    4150 3450
@@
 SCK
 $Comp
-L GND #PWR05
+L GND #PWR04
 U 1 1 56D7102B
 P 9800 2450
-F 0 "#PWR05" H 9800 2200 50  0001 C CNN
+F 0 "#PWR04" H 9800 2200 50  0001 C CNN
 F 1 "GND" H 9800 2300 50  0000 C CNN
 F 2 "" H 9800 2450 50  0000 C CNN
@@
 RADIO_DATA
 $Comp
-L GND #PWR06
+L GND #PWR05
 U 1 1 56D83AA4
 P 9400 3550
-F 0 "#PWR06" H 9400 3300 50  0001 C CNN
+F 0 "#PWR05" H 9400 3300 50  0001 C CNN
 F 1 "GND" H 9400 3400 50  0000 C CNN
 F 2 "" H 9400 3550 50  0000 C CNN
@@
 $EndComp
 $Comp
-L GND #PWR07
+L GND #PWR06
 U 1 1 56D83C01
 P 3350 2150
-F 0 "#PWR07" H 3350 1900 50  0001 C CNN
+F 0 "#PWR06" H 3350 1900 50  0001 C CNN
 F 1 "GND" H 3350 2000 50  0000 C CNN
 F 2 "" H 3350 2150 50  0000 C CNN
@@
 	8600 3850 8600 5950
 Wire Wire Line
-	8600 5050 7600 5050
+	7600 5050 9650 5050
 Connection ~ 8000 3850
 Wire Wire Line
@@
 F 0 "R3" V 5230 3500 50  0000 C CNN
 F 1 "100K" V 5150 3500 50  0000 C CNN
-F 2 "Resistors_SMD:R_1206_HandSoldering" V 5080 3500 50  0001 C CNN
+F 2 "Resistors_SMD:R_0805_HandSoldering" V 5080 3500 50  0001 C CNN
 F 3 "" H 5150 3500 50  0000 C CNN
 	1    5150 3500
@@
 F 0 "R4" V 4830 5800 50  0000 C CNN
 F 1 "100K" V 4750 5800 50  0000 C CNN
-F 2 "Resistors_SMD:R_1206_HandSoldering" V 4680 5800 50  0001 C CNN
+F 2 "Resistors_SMD:R_0805_HandSoldering" V 4680 5800 50  0001 C CNN
 F 3 "" H 4750 5800 50  0000 C CNN
 	1    4750 5800
@@
 F 0 "C3" H 8275 5450 50  0000 L CNN
 F 1 "0.1uf" H 8275 5250 50  0000 L CNN
-F 2 "Capacitors_SMD:C_1206_HandSoldering" H 8288 5200 50  0001 C CNN
+F 2 "Capacitors_SMD:C_0805_HandSoldering" H 8288 5200 50  0001 C CNN
 F 3 "" H 8250 5350 50  0000 C CNN
 	1    8250 5350
@@
 Connection ~ 8250 5050
 $Comp
-L GND #PWR08
+L GND #PWR07
 U 1 1 56D9DFFD
 P 8250 5500
-F 0 "#PWR08" H 8250 5250 50  0001 C CNN
+F 0 "#PWR07" H 8250 5250 50  0001 C CNN
 F 1 "GND" H 8250 5350 50  0000 C CNN
 F 2 "" H 8250 5500 50  0000 C CNN
@@
 F 0 "SW1" H 6100 1700 50  0000 C CNN
 F 1 "Power Switch" H 6150 1400 50  0000 C CNN
-F 2 "Buttons_Switches_ThroughHole:SW_Micro_SPST_Angled" H 6300 1550 50  0001 C CNN
+F 2 "Buttons_Switches_ThroughHole:SW_Micro_SPST" H 6300 1550 50  0001 C CNN
 F 3 "" H 6300 1550 50  0000 C CNN
 	1    6300 1550
@@
 $EndComp
 $Comp
-L GND #PWR09
+L GND #PWR08
 U 1 1 56D9E7B6
 P 6800 1650
-F 0 "#PWR09" H 6800 1400 50  0001 C CNN
+F 0 "#PWR08" H 6800 1400 50  0001 C CNN
 F 1 "GND" H 6800 1500 50  0000 C CNN
 F 2 "" H 6800 1650 50  0000 C CNN
@@
 	1    0    0    -1
 $EndComp
+$Comp
+L POT RV1
+U 1 1 56E809B9
+P 9650 5300
+F 0 "RV1" H 9650 5220 50  0000 C CNN
+F 1 "POT" H 9650 5300 50  0000 C CNN
+F 2 "Potentiometers:Potentiometer_WirePads_largePads" H 9650 5300 50  0001 C CNN
+F 3 "" H 9650 5300 50  0000 C CNN
+	1    9650 5300
+	0    -1   -1   0
+$EndComp
+$Comp
+L GND #PWR09
+U 1 1 56E80AFC
+P 9650 5750
+F 0 "#PWR09" H 9650 5500 50  0001 C CNN
+F 1 "GND" H 9650 5600 50  0000 C CNN
+F 2 "" H 9650 5750 50  0000 C CNN
+F 3 "" H 9650 5750 50  0000 C CNN
+	1    9650 5750
+	1    0    0    -1
+$EndComp
+$Comp
+L VCC #PWR010
+U 1 1 56E80BFE
+P 6800 1050
+F 0 "#PWR010" H 6800 900 50  0001 C CNN
+F 1 "VCC" H 6800 1200 50  0000 C CNN
+F 2 "" H 6800 1050 50  0000 C CNN
+F 3 "" H 6800 1050 50  0000 C CNN
+	1    6800 1050
+	1    0    0    -1
+$EndComp
+Wire Wire Line
+	9650 5050 9650 5150
+$Comp
+L R R5
+U 1 1 56E80FD3
+P 9650 5600
+F 0 "R5" V 9730 5600 50  0000 C CNN
+F 1 "100K" V 9650 5600 50  0000 C CNN
+F 2 "Resistors_SMD:R_0805_HandSoldering" V 9580 5600 50  0001 C CNN
+F 3 "" H 9650 5600 50  0000 C CNN
+	1    9650 5600
+	1    0    0    -1
+$EndComp
+Text Label 4300 5350 0    60   ~ 0
+ADC3
+Text Label 9200 5300 0    60   ~ 0
+ADC3
+Wire Wire Line
+	9500 5300 9200 5300
+Wire Wire Line
+	4900 5350 4300 5350
+$Comp
+L Q_PMOS_GSD Q2
+U 1 1 56E815FA
+P 6450 2450
+F 0 "Q2" H 6750 2500 50  0000 R CNN
+F 1 "Q_PMOS_GSD" H 7100 2400 50  0000 R CNN
+F 2 "TO_SOT_Packages_SMD:SOT-23_Handsoldering" H 6650 2550 50  0001 C CNN
+F 3 "" H 6450 2450 50  0000 C CNN
+	1    6450 2450
+	1    0    0    -1
+$EndComp
+$Comp
+L Q_NMOS_GSD Q1
+U 1 1 56E8170A
+P 5450 3150
+F 0 "Q1" H 5750 3200 50  0000 R CNN
+F 1 "Q_NMOS_GSD" H 6100 3100 50  0000 R CNN
+F 2 "TO_SOT_Packages_SMD:SOT-23_Handsoldering" H 5650 3250 50  0001 C CNN
+F 3 "" H 5450 3150 50  0000 C CNN
+	1    5450 3150
+	1    0    0    -1
+$EndComp
+$Comp
+L APE8865N-12-HF-3 U1
+U 1 1 56E81B2E
+P 7350 3900
+F 0 "U1" H 7500 3600 50  0000 C CNN
+F 1 "MCP1700T-3302E/TT" H 7350 4100 50  0000 C CNN
+F 2 "TO_SOT_Packages_SMD:SOT-23_Handsoldering" H 7350 4000 50  0000 C CIN
+F 3 "" H 7350 3900 50  0000 C CNN
+	1    7350 3900
+	1    0    0    -1
+$EndComp
