File: kicad/pir/rc_power_sockets.sch (KiCad schematic (older format))
At the start: 32 parts, among them IC1 ATTINY85, J1 PIR, J2 433MHZ, J3 433MHZ, P1 ICSP, P2 ALT_PWR, Q1 NMOS, Q2 PMOS, SW1 SWITCH_INV, U1 MCP1755ST-3302E/DB

Commit message: Tiny logo
Parts:
- C4: footprint (none) -> Capacitors_SMD:C_0805_HandSoldering
Changed lines of the file:
@@
 $EndComp
 $Comp
-L GND #PWR11
+L GND #PWR01
 U 1 1 56D4B298
 P 7350 4400
-F 0 "#PWR11" H 7350 4150 50  0001 C CNN
+F 0 "#PWR01" H 7350 4150 50  0001 C CNN
 F 1 "GND" H 7350 4250 50  0000 C CNN
 F 2 "" H 7350 4400 50  0000 C CNN
@@
 $EndComp
 $Comp
-L GND #PWR9
+L GND #PWR02
 U 1 1 56D4D563
 P 5550 3800
-F 0 "#PWR9" H 5550 3550 50  0001 C CNN
+F 0 "#PWR02" H 5550 3550 50  0001 C CNN
 F 1 "GND" H 5550 3650 50  0000 C CNN
 F 2 "" H 5550 3800 50  0000 C CNN
@@
 $EndComp
 $Comp
-L GND #PWR13
+L GND #PWR03
 U 1 1 56D4E393
 P 7600 5550
-F 0 "#PWR13" H 7600 5300 50  0001 C CNN
+F 0 "#PWR03" H 7600 5300 50  0001 C CNN
 F 1 "GND" H 7600 5400 50  0000 C CNN
 F 2 "" H 7600 5550 50  0000 C CNN
@@
 SCK
 $Comp
-L GND #PWR16
+L GND #PWR04
 U 1 1 56D7102B
 P 8450 2400
-F 0 "#PWR16" H 8450 2150 50  0001 C CNN
+F 0 "#PWR04" H 8450 2150 50  0001 C CNN
 F 1 "GND" H 8450 2250 50  0000 C CNN
 F 2 "" H 8450 2400 50  0000 C CNN
@@
 RADIO_DATA
 $Comp
-L GND #PWR21
+L GND #PWR05
 U 1 1 56D83AA4
 P 9400 3550
-F 0 "#PWR21" H 9400 3300 50  0001 C CNN
+F 0 "#PWR05" H 9400 3300 50  0001 C CNN
 F 1 "GND" H 9400 3400 50  0000 C CNN
 F 2 "" H 9400 3550 50  0000 C CNN
@@
 $EndComp
 $Comp
-L GND #PWR8
+L GND #PWR06
 U 1 1 56D83C01
 P 3350 2150
-F 0 "#PWR8" H 3350 1900 50  0001 C CNN
+F 0 "#PWR06" H 3350 1900 50  0001 C CNN
 F 1 "GND" H 3350 2000 50  0000 C CNN
 F 2 "" H 3350 2150 50  0000 C CNN
@@
 $EndComp
 $Comp
-L GND #PWR15
+L GND #PWR07
 U 1 1 56D9DFFD
 P 8250 5500
-F 0 "#PWR15" H 8250 5250 50  0001 C CNN
+F 0 "#PWR07" H 8250 5250 50  0001 C CNN
 F 1 "GND" H 8250 5350 50  0000 C CNN
 F 2 "" H 8250 5500 50  0000 C CNN
@@
 $EndComp
 $Comp
-L GND #PWR19
+L GND #PWR08
 U 1 1 56E80AFC
 P 9350 5200
-F 0 "#PWR19" H 9350 4950 50  0001 C CNN
+F 0 "#PWR08" H 9350 4950 50  0001 C CNN
 F 1 "GND" H 9350 5050 50  0000 C CNN
 F 2 "" H 9350 5200 50  0000 C CNN
@@
 RADIO_DATA
 $Comp
-L GND #PWR20
+L GND #PWR09
 U 1 1 56EEFB0C
 P 9400 2900
-F 0 "#PWR20" H 9400 2650 50  0001 C CNN
+F 0 "#PWR09" H 9400 2650 50  0001 C CNN
 F 1 "GND" H 9400 2750 50  0000 C CNN
 F 2 "" H 9400 2900 50  0000 C CNN
@@
 $EndComp
 $Comp
-L GND #PWR6
+L GND #PWR010
 U 1 1 56F02CD0
 P 1700 1300
-F 0 "#PWR6" H 1700 1050 50  0001 C CNN
+F 0 "#PWR010" H 1700 1050 50  0001 C CNN
 F 1 "GND" H 1700 1150 50  0000 C CNN
 F 2 "" H 1700 1300 50  0000 C CNN
@@
 $EndComp
 $Comp
-L GND #PWR7
+L GND #PWR011
 U 1 1 56F02EF0
 P 2150 1300
-F 0 "#PWR7" H 2150 1050 50  0001 C CNN
+F 0 "#PWR011" H 2150 1050 50  0001 C CNN
 F 1 "GND" H 2150 1150 50  0000 C CNN
 F 2 "" H 2150 1300 50  0000 C CNN
@@
 $EndComp
 $Comp
-L GND #PWR1
+L GND #PWR012
 U 1 1 56F02F76
 P 850 1300
-F 0 "#PWR1" H 850 1050 50  0001 C CNN
+F 0 "#PWR012" H 850 1050 50  0001 C CNN
 F 1 "GND" H 850 1150 50  0000 C CNN
 F 2 "" H 850 1300 50  0000 C CNN
@@
 $EndComp
 $Comp
-L GND #PWR3
+L GND #PWR013
 U 1 1 56F02F82
 P 1300 1300
-F 0 "#PWR3" H 1300 1050 50  0001 C CNN
+F 0 "#PWR013" H 1300 1050 50  0001 C CNN
 F 1 "GND" H 1300 1150 50  0000 C CNN
 F 2 "" H 1300 1300 50  0000 C CNN
@@
 	5550 950  5550 1500
 $Comp
-L GND #PWR12
+L GND #PWR014
 U 1 1 56F5CBEA
 P 7450 1650
-F 0 "#PWR12" H 7450 1400 50  0001 C CNN
+F 0 "#PWR014" H 7450 1400 50  0001 C CNN
 F 1 "GND" H 7450 1500 50  0000 C CNN
 F 2 "" H 7450 1650 50  0000 C CNN
@@
 	2150 5050 1900 5050
 $Comp
-L GND #PWR4
+L GND #PWR015
 U 1 1 56F5DB12
 P 1500 5200
-F 0 "#PWR4" H 1500 4950 50  0001 C CNN
+F 0 "#PWR015" H 1500 4950 50  0001 C CNN
 F 1 "GND" H 1500 5050 50  0000 C CNN
 F 2 "" H 1500 5200 50  0000 C CNN
@@
 Connection ~ 7350 4050
 $Comp
-L VCC #PWR17
+L VCC #PWR016
 U 1 1 56F7F5C9
 P 8600 950
-F 0 "#PWR17" H 8600 800 50  0001 C CNN
+F 0 "#PWR016" H 8600 800 50  0001 C CNN
 F 1 "VCC" H 8600 1100 50  0000 C CNN
 F 2 "" H 8600 950 50  0000 C CNN
@@
 $EndComp
 $Comp
-L GND #PWR18
+L GND #PWR017
 U 1 1 56F7F83F
 P 8600 1050
-F 0 "#PWR18" H 8600 800 50  0001 C CNN
+F 0 "#PWR017" H 8600 800 50  0001 C CNN
 F 1 "GND" H 8600 900 50  0000 C CNN
 F 2 "" H 8600 1050 50  0000 C CNN
@@
 $EndComp
 $Comp
-L GND #PWR2
+L GND #PWR018
 U 1 1 56F8174A
 P 1100 2100
-F 0 "#PWR2" H 1100 1850 50  0001 C CNN
+F 0 "#PWR018" H 1100 1850 50  0001 C CNN
 F 1 "GND" H 1100 1950 50  0000 C CNN
 F 2 "" H 1100 2100 50  0000 C CNN
@@
 $EndComp
 $Comp
-L GND #PWR5
+L GND #PWR019
 U 1 1 56F817AF
 P 1550 2100
-F 0 "#PWR5" H 1550 1850 50  0001 C CNN
+F 0 "#PWR019" H 1550 1850 50  0001 C CNN
 F 1 "GND" H 1550 1950 50  0000 C CNN
 F 2 "" H 1550 2100 50  0000 C CNN
@@
 	6700 850  6550 850
 $Comp
-L GND #PWR10
+L GND #PWR020
 U 1 1 56FBCCBF
 P 6550 1050
-F 0 "#PWR10" H 6550 800 50  0001 C CNN
+F 0 "#PWR020" H 6550 800 50  0001 C CNN
 F 1 "GND" H 6550 900 50  0000 C CNN
 F 2 "" H 6550 1050 50  0000 C CNN
@@
 F 0 "C4" H 8225 1350 50  0000 L CNN
 F 1 "10uF" H 8225 1150 50  0000 L CNN
-F 2 "" H 8238 1100 50  0000 C CNN
+F 2 "Capacitors_SMD:C_0805_HandSoldering" H 8238 1100 50  0001 C CNN
 F 3 "" H 8200 1250 50  0000 C CNN
 	1    8200 1250
@@
 Connection ~ 8200 950
 $Comp
-L GND #PWR14
+L GND #PWR021
 U 1 1 57C751C5
 P 8200 1400
-F 0 "#PWR14" H 8200 1150 50  0001 C CNN
+F 0 "#PWR021" H 8200 1150 50  0001 C CNN
 F 1 "GND" H 8200 1250 50  0000 C CNN
 F 2 "" H 8200 1400 50  0000 C CNN
